File: kicad/cubesatsim_solar.kicad_pcb (KiCad board)
At the start: 2 copper layers, 71.3 x 69.8 mm, 28 parts, among them J1 Sensor Inputs, J10 INA219 Sensor Board, J11 INA219 Sensor Board, J12 INA219 Sensor Board, J2 Battery In/Out, J3 Vdc In, J4 Vout to MoPOWER, J5 RBF Switch, J6 Expansion Interface, J7 INA219 Sensor Board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

Commit message: vB2 PCB Submitted to PCB Way
Parts:
- removed the GPIO at (137.4, 74.8)
- added GPIO: GPIO Male Extra Long (19mm) 20x2 Header Pins, Connector_PinHeader_2.54mm:PinHeader_2x20_P2.54mm_Vertical, F.Cu at (113.3, 76.1)
- added J17: , 35RAPC4BH3:SWITCHCRAFT_35RAPC4BH3, F.Cu at (175.8, 83.7)
- D1, D2, D3, D4, D5: value D -> 1N5817
- J3, J4: footprint Connector_PinHeader_2.54mm:PinHeader_1x02_P2.54mm_Vertical -> Connector_Wire:SolderWirePad_1x02_P3.81mm_Drill1.2mm
- moved J5 17.0 mm to (169.7, 92.3), turned to 90 degrees
- moved J3 4.32 mm to (173.0, 103.5), turned to 270 degrees
- moved J4 4.06 mm to (173.0, 95.9), turned to 270 degrees
- moved OUT- 0.25 mm to (161.6, 101.7)
Routing:
- net GND: track 228.2 -> 140.9 mm
- net Net-(J13-Pad1): track 86.0 -> 64.0 mm
- net Net-(J15-Pad1): track 12.7 -> 26.8 mm
- net Net-(J17-Pad1): track 14.3 -> 24.7 mm
- net Net-(J17-Pad5): track 9.56 -> 19.9 mm
- net Net-(D1-Pad1): track 84.9 -> 76.2 mm
- added copper zone on F.Cu, net GND
Other:
- board size 71.3 x 69.8 mm -> 77.2 x 69.8 mm
- board text added: "AMSAT® CubeSat Simulator Solar Power Board vB2 KU2Y"
- board text removed: "AMSAT® CubeSat Simulator Solar Power Board vB1 by KU2Y"

Commit message: kicad files for vB3 PCB
Parts:
- removed GPIO: GPIO Male Extra Long (19mm) 20x2 Header Pins, Connector_PinHeader_2.54mm:PinHeader_2x20_P2.54mm_Vertical
- removed IN+: IN+, Connector_PinSocket_2.54mm:PinSocket_1x01_P2.54mm_Vertical
- removed IN-: IN-, Connector_PinSocket_2.54mm:PinSocket_1x01_P2.54mm_Vertical
- removed J5: RBF Switch, Connector_PinHeader_2.54mm:PinHeader_1x05_P2.54mm_Vertical
- removed OUT+: OUT+, Connector_PinSocket_2.54mm:PinSocket_1x01_P2.54mm_Vertical
- removed OUT-: OUT-, Connector_PinSocket_2.54mm:PinSocket_1x01_P2.54mm_Vertical
- added D6: 1N5817, Diode_THT:D_DO-41_SOD81_P3.81mm_Vertical_AnodeUp, F.Cu at (167.2, 106.8)
- added D7: LED, Diode_THT:D_DO-41_SOD81_P3.81mm_Vertical_AnodeUp, F.Cu at (171.5, 126.1)
- added J13: INA219 Sensor Board, Connector_PinHeader_2.54mm:PinHeader_1x06_P2.54mm_Vertical, F.Cu at (121.7, 113.1)
- added J14: IN-, Connector_PinSocket_2.54mm:PinSocket_1x01_P2.54mm_Vertical, F.Cu at (120.9, 101.7)
- added J15: OUT+, Connector_PinSocket_2.54mm:PinSocket_1x01_P2.54mm_Vertical, F.Cu at (161.6, 83.9)
- added J16: OUT-, Connector_PinSocket_2.54mm:PinSocket_1x01_P2.54mm_Vertical, F.Cu at (161.6, 101.7)
- added P3: GPIO Male Extra Long (19mm) 20x2 Header Pins, Connector_PinHeader_2.54mm:PinHeader_2x20_P2.54mm_Vertical, F.Cu at (113.3, 76.0)
- added R3: 220, Resistor_THT:R_Axial_DIN0207_L6.3mm_D2.5mm_P5.08mm_Vertical, F.Cu at (171.5, 118.5)
- J1: value Sensor Inputs -> PJ-037AH; footprint Connector_PinHeader_2.54mm:PinHeader_1x10_P2.54mm_Vertical -> PJ-037AH:CUI_PJ-037AH
- J17: value (none) -> IN+; footprint 35RAPC4BH3:SWITCHCRAFT_35RAPC4BH3 -> Connector_PinSocket_2.54mm:PinSocket_1x01_P2.54mm_Vertical
- J2: value Battery In/Out -> CONN_01X14; footprint Connector_PinHeader_2.54mm:PinHeader_1x02_P2.54mm_Vertical -> Connector_PinSocket_2.54mm:PinSocket_1x14_P2.54mm_Vertical
- J3: value Vdc In -> 35RAPC4BH3; footprint Connector_Wire:SolderWirePad_1x02_P3.81mm_Drill1.2mm -> 35RAPC4BH3:SWITCHCRAFT_35RAPC4BH3
- J4: footprint Connector_Wire:SolderWirePad_1x02_P3.81mm_Drill1.2mm -> Connector_PinSocket_2.54mm:PinSocket_2x01_P2.54mm_Vertical
- moved J17 54.9 mm to (120.9, 83.9), turned to 0 degrees
- moved J3 20.0 mm to (175.8, 83.7), turned to 180 degrees
- moved J2 14.7 mm to (175.3, 127.6)
- moved D1 8.76 mm to (129.1, 106.8)
- moved D2 6.48 mm to (136.7, 106.8)
- moved J1 5.95 mm to (169.2, 134.0), turned to 0 degrees
- moved J4 4.89 mm to (175.3, 91.5), turned to 0 degrees
- moved D3 4.00 mm to (144.0, 106.8)
- moved D4 1.78 mm to (151.9, 106.9)
- moved J7 1.30 mm to (162.6, 121.5)
- moved J8 1.30 mm to (153.8, 121.5)
- moved J9 1.30 mm to (144.8, 121.5)
- moved J10 1.30 mm to (135.7, 121.3)
- moved J11 1.30 mm to (126.5, 121.5)
- moved J12 1.30 mm to (117.4, 121.3)
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Connections:
- net X+Out renamed +X_Out
- net X-Out renamed -X_Out
- net Y+Out renamed +Y_Out
- net Y-Out renamed -Y_Out
- net Z+Out renamed +Z_Out
- J1 pad 1: X+In -> Net-(J1-Pad1)
- J11 pad 1: X-In -> -X_In
- J12 pad 1: Y-In -> -Y_In
- J2 pad 1: VbattIn -> +X_In
- J2 pad 2: VbattOut -> GND
- J3 pad 1: Net-(J17-Pad1) -> Net-(J1-Pad1)
- J3 pad 2: GND -> Net-(J17-Pad1)
- J4 pad 1: Net-(J17-Pad5) -> Net-(J3-Pad5)
- J7 pad 1: X+In -> +X_In
- J8 pad 1: Y+In -> +Y_In
- J9 pad 1: Z+In -> +Z_In
Routing:
- net Net-(D7-Pad1): track 0.00 -> 93.8 mm, vias 0 -> 2
- net -Y_In: track 0.00 -> 70.1 mm, vias 0 -> 2
- net -Z_In: track 0.00 -> 65.1 mm, vias 0 -> 1
- net -X_In: track 0.00 -> 64.3 mm, vias 0 -> 2
- net Net-(J13-Pad1): track 64.0 -> 0.00 mm
- net Y-In: track 58.8 -> 0.00 mm
- net Net-(J1-Pad1): track 0.00 -> 58.4 mm, vias 0 -> 1
- net -Z_Out: track 0.00 -> 57.6 mm, vias 0 -> 1
- net X-In: track 50.1 -> 0.00 mm
- net Net-(J17-Pad1): track 24.7 -> 66.8 mm, vias 0 -> 2
- net Net-(D1-Pad1): track 76.2 -> 115.9 mm
- net +Z_In: track 0.00 -> 36.0 mm, vias 0 -> 1
- net Z+In: track 34.3 -> 0.00 mm, vias 1 -> 0
- net Y+In: track 30.4 -> 0.00 mm, vias 1 -> 0
- net +3V3: track 153.2 -> 182.8 mm, vias 2 -> 3
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Other:
- board text added: "+X"
- board text added: "+Y"
- board text added: "+Z"
- board text added: "-X"
- board text added: "-Y"
- board text added: "-Z"
- board text added: "3.3"
- board text added: "5V"
- board text added: "AMSAT® CubeSat Simulator Solar Power Board vB3"
- board text added: "DC in"
- board text added: "GND"
- board text added: "IN+"
- board text added: "IN-"
- board text added: "KU2Y"
- board text added: "OUT+"
- board text added: "OUT-"
- board text added: "RBF Switch"
- board text added: "SCL"
- board text added: "SDA"
- board text added: "Vout"
- board text added: "batt"
- board text removed: "AMSAT® CubeSat Simulator Solar Power Board vB2 KU2Y"
