File: kicad/cubesatsim_solar.sch (KiCad schematic (older format))
At the start: 23 parts, among them J1 Sensor Inputs, J10 INA219 Sensor Board, J11 INA219 Sensor Board, J12 INA219 Sensor Board, J13 3.5mm TRS Audio Jack with 2 S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, J14 RBF connector, J2 Battery In/Out, J3 Vout to MoPOWER, J4 Vdc In, J5 RBF Switch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

Commit message: Add files via upload
Changed lines of the file:
@@
 EESchema Schematic File Version 4
+LIBS:cubesatsim_solar-cache
 EELAYER 26 0
 EELAYER END
@@
 P 2300 2700
 F 0 "P3" H 1200 4650 60  0000 C CNN
-F 1 "Male Extra Long (19mm) 20x2 Header Pins" H 2050 1175 60  0000 C CNN
+F 1 "Male Extra Long (19mm) 20x2 Header Pins" H 2075 900 60  0000 C CNN
 F 2 "w_conn_strip:vasch_strip_20x2" H 2300 2700 60  0001 C CNN
 F 3 "" H 2300 2700 60  0000 C CNN
@@
 Wire Wire Line
 	8050 1875 8050 2700
+Text Label 1975 4375 0    50   ~ 0
+Raspberry Pi GPIO Connector
 $EndSCHEMATC

Commit message: Add files via upload
Parts:
- D1, D2, D3, D4, D5: value D -> 1N5817
- P3: value Male Extra Long (19mm) 20x2 Header Pins -> Raspberry Pi GPIO Connector
Other:
- note added: "Between NiMH battery and MoPower Board"
- note added: "Boost Converter trim pot adjusted to give 15V output at maximum solar panel voltage input."
- note added: "INA219 boards are mounted vertically with 45 degree 5x1 pins"
- note added: "Male Extra Long (19mm) 20x2 Header Pins"
- note added: "To 5.5mm x 2.1mm"
- note added: "With RBF switch inserted (3.5mm jack plugged in), \nVout to MoPower comes from the Vdc in barrel jack\nthrough 3.5mm plug that has jumper between 3 and 1 \n(center and outer). Solar panels are isolated from the \ninput to the boost converter through the switch.\n"
- note added: "With the RBF switch removed, the solar panels are \nconnected to the boost converter input and the \noutput of the boost converter is connected to \nthe Vout to the MoPower board."
- note added: "female barrel jack"
Changed lines of the file:
@@
 Sheet 1 1
 Title "AMSAT CubeSat Simulator Solar Panel Board"
-Date ""
+Date "December 8, 2018"
 Rev "Beta1"
 Comp "See https://github.com/alanbjohnston/cubesatsim"
@@
 P 5350 2425
 F 0 "D1" H 5350 2641 50  0000 C CNN
-F 1 "D" H 5350 2550 50  0000 C CNN
+F 1 "1N5817" H 5350 2550 50  0000 C CNN
 F 2 "Diode_THT:D_DO-41_SOD81_P3.81mm_Vertical_AnodeUp" H 5350 2425 50  0001 C CNN
 F 3 "~" H 5350 2425 50  0001 C CNN
@@
 P 2300 2700
 F 0 "P3" H 1200 4650 60  0000 C CNN
-F 1 "Male Extra Long (19mm) 20x2 Header Pins" H 2075 900 60  0000 C CNN
+F 1 "Raspberry Pi GPIO Connector" H 2025 1225 60  0000 C CNN
 F 2 "w_conn_strip:vasch_strip_20x2" H 2300 2700 60  0001 C CNN
 F 3 "" H 2300 2700 60  0000 C CNN
@@
 P 5350 2750
 F 0 "D2" H 5350 2966 50  0000 C CNN
-F 1 "D" H 5350 2875 50  0000 C CNN
+F 1 "1N5817" H 5350 2875 50  0000 C CNN
 F 2 "Diode_THT:D_DO-41_SOD81_P3.81mm_Vertical_AnodeUp" H 5350 2750 50  0001 C CNN
 F 3 "~" H 5350 2750 50  0001 C CNN
@@
 P 5350 3100
 F 0 "D3" H 5350 3316 50  0000 C CNN
-F 1 "D" H 5350 3225 50  0000 C CNN
+F 1 "1N5817" H 5350 3225 50  0000 C CNN
 F 2 "Diode_THT:D_DO-41_SOD81_P3.81mm_Vertical_AnodeUp" H 5350 3100 50  0001 C CNN
 F 3 "~" H 5350 3100 50  0001 C CNN
@@
 P 5350 3425
 F 0 "D4" H 5350 3641 50  0000 C CNN
-F 1 "D" H 5350 3550 50  0000 C CNN
+F 1 "1N5817" H 5350 3550 50  0000 C CNN
 F 2 "Diode_THT:D_DO-41_SOD81_P3.81mm_Vertical_AnodeUp" H 5350 3425 50  0001 C CNN
 F 3 "~" H 5350 3425 50  0001 C CNN
@@
 P 5350 3775
 F 0 "D5" H 5350 3991 50  0000 C CNN
-F 1 "D" H 5350 3900 50  0000 C CNN
+F 1 "1N5817" H 5350 3900 50  0000 C CNN
 F 2 "Diode_THT:D_DO-41_SOD81_P3.81mm_Vertical_AnodeUp" H 5350 3775 50  0001 C CNN
 F 3 "~" H 5350 3775 50  0001 C CNN
@@
 Wire Wire Line
 	6700 1775 8925 1775
-Text Label 4800 3975 0    50   ~ 0
-1N5817 Schottky Barrier Diodes
 $Comp
 L pihat_template-rescue:BoostConverter-New_Library U1
@@
 Wire Wire Line
 	6700 1775 6700 2700
-Text Label 6150 3400 0    50   ~ 0
-Boost Converter trim pot adjusted to give 15V output at maximum solar panel voltage input.
 $Comp
 L pihat_template-rescue:Audio-Jack-3_2Switches-conn2 J13
@@
 P 9050 1025
 F 0 "J13" H 8762 1002 50  0000 R CNN
-F 1 "3.5mm TRS Audio Jack with 2 Switches" H 8762 1093 50  0000 R CNN
+F 1 "3.5mm TRS Audio Jack with 2 Switches" H 9850 725 50  0000 R CNN
 F 2 "" H 9300 1125 50  0001 C CNN
 F 3 "" H 9300 1125 50  0001 C CNN
@@
 	-1   0    0    -1
 $EndComp
-Text Label 5700 6600 0    50   ~ 0
-INA219 boards are mounted vertically with 45 degree 5x1 pins
-Text Label 5825 1325 0    50   ~ 0
-3.5mm plug for RBF switch has jumper between 3 and 1 (center and outer)
 Wire Wire Line
 	9475 1975 9850 1975
@@
 Text Label 9550 5450 0    50   ~ 0
 To Solar Panels
-Text Label 8500 6625 0    50   ~ 0
-Between NiMH battery and MoPower Board
-Text Label 9475 2450 0    50   ~ 0
-female barrel jack
-Text Label 9475 2350 0    50   ~ 0
-To 5.5mm x 2.1mm
 Text Label 12250 10925 0    50   ~ 0
 AMSAT CubeSat Simulator Solar Power Board
@@
 Wire Wire Line
 	8050 1875 8050 2700
-Text Label 1975 4375 0    50   ~ 0
-Raspberry Pi GPIO Connector
+Text Notes 9475 2350 0    50   ~ 0
+To 5.5mm x 2.1mm
+Text Notes 9475 2450 0    50   ~ 0
+female barrel jack
+Text Notes 6050 1450 0    50   ~ 0
+With the RBF switch removed, the solar panels are \nconnected to the boost converter input and the \noutput of the boost converter is connected to \nthe Vout to the MoPower board.
+Text Notes 6150 3400 0    50   ~ 0
+Boost Converter trim pot adjusted to give 15V output at maximum solar panel voltage input.
+Text Notes 8500 6625 0    50   ~ 0
+Between NiMH battery and MoPower Board
+Text Notes 5700 6600 0    50   ~ 0
+INA219 boards are mounted vertically with 45 degree 5x1 pins
+Text Notes 1700 4325 0    50   ~ 0
+Male Extra Long (19mm) 20x2 Header Pins
+Text Notes 6050 1025 0    50   ~ 0
+With RBF switch inserted (3.5mm jack plugged in), \nVout to MoPower comes from the Vdc in barrel jack\nthrough 3.5mm plug that has jumper between 3 and 1 \n(center and outer). Solar panels are isolated from the \ninput to the boost converter through the switch.\n
 $EndSCHEMATC

Commit message: Preliminary PCB Design
Connections:
- net SCL_0 renamed SCL_3
- net SDA_0 renamed SDA_3
Other:
- note added: "INA219 boards are mounted vertically with 90 degree 5x1 header pins"
- note removed: "INA219 boards are mounted vertically with 45 degree 5x1 pins"
- moved on the sheet: J10, J11
Changed lines of the file:
@@
 Sheet 1 1
 Title "AMSAT CubeSat Simulator Solar Panel Board"
-Date "December 8, 2018"
-Rev "Beta1"
+Date "December 13, 2018"
+Rev "Beta1.1"
 Comp "See https://github.com/alanbjohnston/cubesatsim"
 Comment1 ""
@@
 	7325 5475 7325 5450
 Text GLabel 975  3100 0    50   Input ~ 0
-SDA_0
+SDA_3
 Text GLabel 975  3000 0    50   Input ~ 0
-SCL_0
+SCL_3
 $Comp
 L pihat_template-rescue:Raspberry_Pi_+_Conn-pihat_template-rescue P3
@@
 Wire Wire Line
 	1025 3000 1200 3000
-Text GLabel 7450 5750 0    50   Input ~ 0
+Text GLabel 2575 4950 0    50   Input ~ 0
 VbattIn
-Text GLabel 7450 5850 0    50   Input ~ 0
+Text GLabel 2575 5050 0    50   Input ~ 0
 VbattOut
-Text GLabel 7450 5950 0    50   Input ~ 0
+Text GLabel 2575 5150 0    50   Input ~ 0
 SDA_1
-Text GLabel 7450 6050 0    50   Input ~ 0
+Text GLabel 2575 5250 0    50   Input ~ 0
 SCL_1
 $Comp
 L pihat_template-rescue:GND-power #PWR05
 U 1 1 5BF9E33A
-P 6900 6250
-F 0 "#PWR05" H 6900 6000 50  0001 C CNN
-F 1 "GND" H 6905 6077 50  0000 C CNN
-F 2 "" H 6900 6250 50  0001 C CNN
-F 3 "" H 6900 6250 50  0001 C CNN
-	1    6900 6250
-	1    0    0    -1
-$EndComp
-Wire Wire Line
-	6900 6250 6900 6150
-Wire Wire Line
-	6900 6150 7450 6150
+P 2025 5450
+F 0 "#PWR05" H 2025 5200 50  0001 C CNN
+F 1 "GND" H 2030 5277 50  0000 C CNN
+F 2 "" H 2025 5450 50  0001 C CNN
+F 3 "" H 2025 5450 50  0001 C CNN
+	1    2025 5450
+	1    0    0    -1
+$EndComp
+Wire Wire Line
+	2025 5450 2025 5350
+Wire Wire Line
+	2025 5350 2575 5350
 $Comp
 L pihat_template-rescue:Conn_01x06_Female-Connector J10
 U 1 1 5BF9E342
-P 7650 5950
-F 0 "J10" H 7678 5926 50  0000 L CNN
-F 1 "INA219 Sensor Board" H 7678 5835 50  0000 L CNN
-F 2 "Connector_PinHeader_2.54mm:PinHeader_1x06_P2.54mm_Vertical" H 7650 5950 50  0001 C CNN
-F 3 "~" H 7650 5950 50  0001 C CNN
-	1    7650 5950
-	1    0    0    -1
-$EndComp
-Wire Wire Line
-	7450 6250 7375 6250
-Wire Wire Line
-	7375 6250 7375 6325
-Wire Wire Line
-	7375 6325 7325 6325
+P 2775 5150
+F 0 "J10" H 2803 5126 50  0000 L CNN
+F 1 "INA219 Sensor Board" H 2803 5035 50  0000 L CNN
+F 2 "Connector_PinHeader_2.54mm:PinHeader_1x06_P2.54mm_Vertical" H 2775 5150 50  0001 C CNN
+F 3 "~" H 2775 5150 50  0001 C CNN
+	1    2775 5150
+	1    0    0    -1
+$EndComp
+Wire Wire Line
+	2575 5450 2500 5450
+Wire Wire Line
+	2500 5450 2500 5525
+Wire Wire Line
+	2500 5525 2450 5525
 $Comp
 L pihat_template-rescue:+3.3V-PiHatAx5043-cache #PWR0101
@@
 $EndComp
 Text GLabel 2200 6875 0    50   Input ~ 0
-SDA_0
+SDA_3
 Text GLabel 2200 6975 0    50   Input ~ 0
-SCL_0
+SCL_3
 Wire Wire Line
 	2275 6875 2200 6875
@@
 L pihat_template-rescue:power_+3.3V-PiHatAx5043-cache #PWR0115
 U 1 1 5BFB928B
-P 7325 6325
-F 0 "#PWR0115" H 7325 6175 50  0001 C CNN
-F 1 "power_+3.3V" H 7350 6275 50  0000 C CNN
-F 2 "" H 7325 6325 50  0001 C CNN
-F 3 "" H 7325 6325 50  0001 C CNN
-	1    7325 6325
+P 2450 5525
+F 0 "#PWR0115" H 2450 5375 50  0001 C CNN
+F 1 "power_+3.3V" H 2475 5475 50  0000 C CNN
+F 2 "" H 2450 5525 50  0001 C CNN
+F 3 "" H 2450 5525 50  0001 C CNN
+	1    2450 5525
 	1    0    0    -1
 $EndComp
 Text Notes 7750 5350 0    50   ~ 0
 I2C Address 0x40
-Text Notes 7750 6200 0    50   ~ 0
+Text Notes 2875 5400 0    50   ~ 0
 I2C Address 0x45
 Text GLabel 5850 4925 0    50   Input ~ 0
@@
 Text Notes 4450 5400 0    50   ~ 0
 I2C Address 0x44\n
-Text GLabel 2450 4925 0    50   Input ~ 0
+Text GLabel 7450 5750 0    50   Input ~ 0
 X-In
-Text GLabel 2450 5025 0    50   Input ~ 0
+Text GLabel 7450 5850 0    50   Input ~ 0
 X-Out
-Text GLabel 2450 5125 0    50   Input ~ 0
-SDA_0
-Text GLabel 2450 5225 0    50   Input ~ 0
-SCL_0
+Text GLabel 7450 5950 0    50   Input ~ 0
+SDA_3
+Text GLabel 7450 6050 0    50   Input ~ 0
+SCL_3
 $Comp
 L pihat_template-rescue:GND-power #PWR0120
 U 1 1 5BFBED52
-P 1900 5425
-F 0 "#PWR0120" H 1900 5175 50  0001 C CNN
-F 1 "GND" H 1905 5252 50  0000 C CNN
-F 2 "" H 1900 5425 50  0001 C CNN
-F 3 "" H 1900 5425 50  0001 C CNN
-	1    1900 5425
-	1    0    0    -1
-$EndComp
-Wire Wire Line
-	1900 5425 1900 5325
-Wire Wire Line
-	1900 5325 2450 5325
+P 6900 6250
+F 0 "#PWR0120" H 6900 6000 50  0001 C CNN
+F 1 "GND" H 6905 6077 50  0000 C CNN
+F 2 "" H 6900 6250 50  0001 C CNN
+F 3 "" H 6900 6250 50  0001 C CNN
+	1    6900 6250
+	1    0    0    -1
+$EndComp
+Wire Wire Line
+	6900 6250 6900 6150
+Wire Wire Line
+	6900 6150 7450 6150
 $Comp
 L pihat_template-rescue:Conn_01x06_Female-Connector J11
 U 1 1 5BFBED5A
-P 2650 5125
-F 0 "J11" H 2678 5101 50  0000 L CNN
-F 1 "INA219 Sensor Board" H 2678 5010 50  0000 L CNN
-F 2 "Connector_PinHeader_2.54mm:PinHeader_1x06_P2.54mm_Vertical" H 2650 5125 50  0001 C CNN
-F 3 "~" H 2650 5125 50  0001 C CNN
-	1    2650 5125
-	1    0    0    -1
-$EndComp
-Wire Wire Line
-	2450 5425 2375 5425
-Wire Wire Line
-	2375 5425 2375 5500
-Wire Wire Line
-	2375 5500 2325 5500
-Wire Wire Line
-	2325 5500 2325 5475
+P 7650 5950
+F 0 "J11" H 7678 5926 50  0000 L CNN
+F 1 "INA219 Sensor Board" H 7678 5835 50  0000 L CNN
+F 2 "Connector_PinHeader_2.54mm:PinHeader_1x06_P2.54mm_Vertical" H 7650 5950 50  0001 C CNN
+F 3 "~" H 7650 5950 50  0001 C CNN
+	1    7650 5950
+	1    0    0    -1
+$EndComp
+Wire Wire Line
+	7450 6250 7375 6250
+Wire Wire Line
+	7375 6250 7375 6325
+Wire Wire Line
+	7375 6325 7325 6325
+Wire Wire Line
+	7325 6325 7325 6300
 $Comp
 L pihat_template-rescue:power_+3.3V-PiHatAx5043-cache #PWR0121
 U 1 1 5BFBED64
-P 2325 5475
-F 0 "#PWR0121" H 2325 5325 50  0001 C CNN
-F 1 "power_+3.3V" H 2275 5400 50  0000 C CNN
-F 2 "" H 2325 5475 50  0001 C CNN
-F 3 "" H 2325 5475 50  0001 C CNN
-	1    2325 5475
-	1    0    0    -1
-$EndComp
-Text Notes 2725 5375 0    50   ~ 0
+P 7325 6300
+F 0 "#PWR0121" H 7325 6150 50  0001 C CNN
+F 1 "power_+3.3V" H 7275 6225 50  0000 C CNN
+F 2 "" H 7325 6300 50  0001 C CNN
+F 3 "" H 7325 6300 50  0001 C CNN
+	1    7325 6300
+	1    0    0    -1
+$EndComp
+Text Notes 7725 6200 0    50   ~ 0
 I2C Address 0x40
 Text GLabel 5800 5775 0    50   Input ~ 0
@@
 Y-Out
 Text GLabel 5800 5975 0    50   Input ~ 0
-SDA_0
+SDA_3
 Text GLabel 5800 6075 0    50   Input ~ 0
-SCL_0
+SCL_3
 $Comp
 L pihat_template-rescue:GND-power #PWR0122
@@
 Between NiMH battery and MoPower Board
 Text Notes 5700 6600 0    50   ~ 0
-INA219 boards are mounted vertically with 45 degree 5x1 pins
+INA219 boards are mounted vertically with 90 degree 5x1 header pins
 Text Notes 1700 4325 0    50   ~ 0
 Male Extra Long (19mm) 20x2 Header Pins

Commit message: Switched J3 and J4 reference in schematic to match PCB
Parts:
- renumbered J4 to J3, J3 to J4
Connections:
- net GND: no longer J3.2 (P2)
Other:
- moved on the sheet: J3, J4
Changed lines of the file:
@@
 Sheet 1 1
 Title "AMSAT CubeSat Simulator Solar Panel Board"
-Date "December 13, 2018"
-Rev "Beta1.1"
+Date "December 15, 2018"
+Rev "Beta1.2"
 Comp "See https://github.com/alanbjohnston/cubesatsim"
-Comment1 ""
+Comment1 "KU2Y"
 Comment2 ""
 Comment3 ""
@@
 $EndComp
 $Comp
-L pihat_template-rescue:CONN_01X02-conn2 J4
+L pihat_template-rescue:CONN_01X02-conn2 J3
 U 1 1 5BF6082F
-P 9125 2350
-F 0 "J4" H 9202 2391 50  0000 L CNN
-F 1 "Vdc In" H 9202 2300 50  0000 L CNN
-F 2 "Connector_PinHeader_2.54mm:PinHeader_1x02_P2.54mm_Vertical" H 9125 2350 50  0001 C CNN
-F 3 "" H 9125 2350 50  0001 C CNN
-	1    9125 2350
-	1    0    0    -1
-$EndComp
-$Comp
-L pihat_template-rescue:CONN_01X02-conn2 J3
-U 1 1 5BF6089F
 P 9125 2700
-F 0 "J3" H 9203 2741 50  0000 L CNN
-F 1 "Vout to MoPOWER" H 9203 2650 50  0000 L CNN
+F 0 "J3" H 9202 2741 50  0000 L CNN
+F 1 "Vdc In" H 9202 2650 50  0000 L CNN
 F 2 "Connector_PinHeader_2.54mm:PinHeader_1x02_P2.54mm_Vertical" H 9125 2700 50  0001 C CNN
 F 3 "" H 9125 2700 50  0001 C CNN
@@
 $EndComp
 $Comp
+L pihat_template-rescue:CONN_01X02-conn2 J4
+U 1 1 5BF6089F
+P 9125 2375
+F 0 "J4" H 9203 2416 50  0000 L CNN
+F 1 "Vout to MoPOWER" H 9203 2325 50  0000 L CNN
+F 2 "Connector_PinHeader_2.54mm:PinHeader_1x02_P2.54mm_Vertical" H 9125 2375 50  0001 C CNN
+F 3 "" H 9125 2375 50  0001 C CNN
+	1    9125 2375
+	1    0    0    -1
+$EndComp
+$Comp
 L pihat_template-rescue:GND-power #PWR0105
 U 1 1 5BF609A2
-P 8925 2400
-F 0 "#PWR0105" H 8925 2150 50  0001 C CNN
-F 1 "GND-power" H 8925 2250 50  0000 C CNN
-F 2 "" H 8925 2400 50  0001 C CNN
-F 3 "" H 8925 2400 50  0001 C CNN
-	1    8925 2400
+P 8950 2750
+F 0 "#PWR0105" H 8950 2500 50  0001 C CNN
+F 1 "GND-power" H 8950 2600 50  0000 C CNN
+F 2 "" H 8950 2750 50  0001 C CNN
+F 3 "" H 8950 2750 50  0001 C CNN
+	1    8950 2750
 	1    0    0    -1
 $EndComp
@@
 L pihat_template-rescue:GND-power #PWR0106
 U 1 1 5BF609DA
-P 8925 2750
-F 0 "#PWR0106" H 8925 2500 50  0001 C CNN
-F 1 "GND-power" H 8930 2577 50  0000 C CNN
-F 2 "" H 8925 2750 50  0001 C CNN
-F 3 "" H 8925 2750 50  0001 C CNN
-	1    8925 2750
-	1    0    0    -1
-$EndComp
-Wire Wire Line
-	8550 2650 8550 1975
+P 8925 2425
+F 0 "#PWR0106" H 8925 2175 50  0001 C CNN
+F 1 "GND-power" H 8875 2300 50  0000 C CNN
+F 2 "" H 8925 2425 50  0001 C CNN
+F 3 "" H 8925 2425 50  0001 C CNN
+	1    8925 2425
+	1    0    0    -1
+$EndComp
+Wire Wire Line
+	8550 2325 8550 1975
 Wire Wire Line
 	8550 1975 8925 1975
 Wire Wire Line
-	8925 2075 8750 2075
-Wire Wire Line
-	8750 2075 8750 2300
-Wire Wire Line
-	8750 2300 8925 2300
+	8925 2075 8625 2075
+Wire Wire Line
+	8625 2075 8625 2650
+Wire Wire Line
+	8625 2650 8925 2650
 Wire Wire Line
 	5500 2425 5625 2425
@@
 	1075 1250 1075 1225
 Wire Wire Line
-	8550 2650 8925 2650
+	8550 2325 8925 2325
 $Comp
 L pihat_template-rescue:+5V-power #PWR0111
@@
 Wire Wire Line
 	8050 1875 8050 2700
-Text Notes 9475 2350 0    50   ~ 0
+Text Notes 9550 2750 0    50   ~ 0
 To 5.5mm x 2.1mm
-Text Notes 9475 2450 0    50   ~ 0
+Text Notes 9575 2850 0    50   ~ 0
 female barrel jack
 Text Notes 6050 1450 0    50   ~ 0
